File: CPU_DEB/V0.10/5vto3v3.sch (KiCad schematic (older format))
At the start: 38 parts, among them Q1 BSS123, Q2 BSS123, Q3 BSS123, Q4 BSS123, U2 74LVCC3245, U3 74LVCC3245, U4 PCA9306, U5 PCA9306, U6 74LVCC3245, U8 LM75A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

Commit message: INIT
Parts:
- removed R11, R12: 2.1k, Resistors_SMD:R_0603, symbol R
- removed R39: 220k, Resistors_SMD:R_0603, symbol R
- removed R49: 10k, Resistors_SMD:R_0603, symbol R
- removed U3: 74LVCC3245, CEN-PCB:SSOP24, symbol 74LVCC3245
- removed U5: PCA9306, f4deb-mod-library:VSSOP-8, symbol PCA9306
- added Q7, Q8: BSS123, TO_SOT_Packages_SMD:SOT-23, symbol BSS123
- added R1, R2: 4.7k, Resistors_SMD:R_0603, symbol R
- added R16, R18: 12k, Resistors_SMD:R_0603, symbol R
- added R17, R19: 22k, Resistors_SMD:R_0603, symbol R
- R13: value 1k -> 12k
- R14: value 1k -> 22k
- R45: value R -> 330
- R46: value R -> 100
Connections:
- net SCL4-5V is gone; now on net U2RX: R13.2
- net SDA4-5V is gone; now on net GND: R14.2
- net U1TX is gone; now on net U6TX: R48.2, U2.6 (A4)
- net U1TX-5V is gone; now on net U6TX-5V: U2.18 (B4)
- net +5V: no longer R13.1, R14.1, R40.1, R41.1, R43.1
- net +5VA: now also R40.1, R41.1, R43.1, RVAR1.3, R1.1, R2.1; no longer RVAR1.1
- net BD0: now also U6.14 (B8); no longer U6.18 (B4)
- net BD1: now also U6.15 (B7); no longer U6.16 (B6)
- net BD2: now also U6.16 (B6); no longer U6.17 (B5)
- net BD3: now also U6.17 (B5); no longer U6.14 (B8)
- net BD4: now also U6.18 (B4); no longer U6.15 (B7)
- net BE: now also U2.21 (B1); no longer U2.19 (B3)
- net BRS: now also U2.19 (B3); no longer U2.20 (B2)
- net BRW: now also U2.20 (B2); no longer U2.21 (B1)
- net D0: now also U6.10 (A8); no longer U6.6 (A4)
- net D1: now also U6.9 (A7); no longer U6.8 (A6)
- net D2: now also U6.8 (A6); no longer U6.7 (A5)
- net D3: now also U6.7 (A5); no longer U6.10 (A8)
- net D4: now also U6.6 (A4); no longer U6.9 (A7)
- net E: now also U2.3 (A1); no longer U2.5 (A3)
- net GND: now also RVAR1.1, Q7.2 (S), Q8.2 (S), R17.2, R19.2; no longer RVAR1.3
- net RS: now also U2.5 (A3); no longer U2.4 (A2)
- net RW: now also U2.4 (A2); no longer U2.3 (A1)
- net U2RX: now also R14.1
- net U2RX-5V: now also R13.1
- net U2TX: now also R51.2, U2.10 (A8); no longer U2.7 (A5)
- net U2TX-5V: now also U2.14 (B8); no longer U2.17 (B5)
- net U5RX: now also R16.2, R17.1
- net U5RX-5V: now also R16.1
- net U6RX: now also R18.2, R19.1
- net U6RX-5V: now also R18.1
- net U6TX: no longer R51.2, U2.10 (A8)
- net U6TX-5V: no longer U2.14 (B8)
- net at U9.1 (OSCI): now also X1.1; no longer X1.2
- net at C12.1, U9.2 (OSCO): now also X1.2; no longer X1.1
- new net OC3: Q7.1 (G)
- new net OC3-5V: Q7.3 (D), R1.2
- new net OC4: Q8.1 (G)
- new net OC4-5V: Q8.3 (D), R2.2
- no-connect marks 15 -> 8
Other:
- note removed: "PORTB => PORTA\n"
- moved on the sheet: Q2, R41, RVAR1
