File: CPU_DEB/V0.10/CPU_DEB.sch (KiCad schematic (older format))
At the start: 37 parts, among them J1 SIL1, J2 SIL1, J3 SIL1, J4 SIL1, J5 RJ12, J6 SIL1, J7 SIL1, K1 CONN_3, K2 CONN_3, K3 CONN_3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

Commit message: INIT
Parts:
- removed D11, D3, D4: LED, LEDs:LED_0603, symbol LED
- removed J1, J2, J3, J4, J6, J7: SIL1, f4deb-mod-library:COLONETTE, symbol SIL1
- removed P11: CONN_2, Connectors_Molex:Molex_KK_6410-02, symbol CONN_2
- removed P2, P6: CONN_4, Connectors_Molex:Molex_KK_6410-04, symbol CONN_4
- removed R1: 1k, Resistors_SMD:R_0603, symbol R
- removed R2: 330, Resistors_SMD:R_0603, symbol R
- removed R44: 3..3k, Resistors_SMD:R_0603, symbol R
- removed S1, S2: SW_DIP_x4, Buttons_Switches_ThroughHole:SW_DIP_x4_Piano, symbol SW_DIP_x4
- added K10, K9: CONN_3, f4deb-mod-library:KK-3-H, symbol CONN_3
- added SW1: SW_DIP_x08, Buttons_Switches_ThroughHole:SW_DIP_x8_Piano, symbol SW_DIP_x08
- K5, K6, K7: footprint f4deb-mod-library:KK-3 -> f4deb-mod-library:KK-3-H
- K8, P10, P8: footprint Connectors_Molex:Molex_KK_6410-02 -> f4deb-mod-library:KK-2-H
- P4, P5, P7: footprint Connectors_Molex:Molex_KK_6410-04 -> f4deb-mod-library:KK-4-H
- P9: value CONN_5 -> CONN_6; footprint Connectors_Molex:Molex_KK_6410-05 -> f4deb-mod-library:KK-6-H; symbol CONN_5 -> CONN_6
Connections:
- wire segments 179 -> 166
- no-connect marks 9 -> 3
Other:
- note added: "S4"
- note added: "S5"
- note added: "UART-5"
- note removed: "FIXATION"
- note removed: "I2C-4"
- moved on the sheet: D1, D2, J5, K1, K2, K3, K4, K5, K6, K7, K8, P1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
