File: CPU_DEB/V0.10/PIC32.sch (KiCad schematic (older format))
At the start: 47 parts, among them Q5 IRFL9014TRPBF, Q6 2N7002, U1 PIC32MX795F512H, U7 24C512

Commit message: INIT
Parts:
- removed D10, D7, D8, D9: LED, LEDs:LED_0603, symbol LED
- removed R16, R17, R18, R19, R26, R27, R28, R29: 10K, Resistors_SMD:R_0603, symbol R
- added R11, R12: 47k, CEN-PCB:SM0603_Resistor, symbol R
- R20, R21, R22, R23, R24, R25: value 10K -> 47k; footprint Resistors_SMD:R_0603 -> CEN-PCB:SM0603_Resistor
- R30, R31, R32, R33: value 3.2k -> 3.3k
- R34, R35, R36, R37: value 1.5k -> 1.2k
Connections:
- net +3V3: now also U1.26 (VDD), R11.1, R12.1; no longer U1.10 (VDD)
- net CAN1: now also R30.1
- net CAN2: now also R31.1
- net CAN3: now also R32.1
- net CAN4: now also R33.1
- net D0: now also U1.2 (ETXD0/PMD6/RE6); no longer U1.60 (ERXD1/PMD0/RE0)
- net D1: now also U1.1 (ETXEN/PMD5/RE5); no longer U1.61 (ERXD0/PMD1/RE1)
- net D2: now also U1.3 (ETXD1/PMD7/RE7); no longer U1.62 (ERXDV/ECRSDV/PMD2/RE2)
- net D3: now also U1.64 (ERXERR/PMD4/RE4); no longer U1.63 (ERXCLK/EREFCLK/PMD3/RE3)
- net D4: now also U1.63 (ERXCLK/EREFCLK/PMD3/RE3); no longer U1.64 (ERXERR/PMD4/RE4)
- net D5: now also U1.62 (ERXDV/ECRSDV/PMD2/RE2); no longer U1.1 (ETXEN/PMD5/RE5)
- net D6: now also U1.61 (ERXD0/PMD1/RE1); no longer U1.2 (ETXD0/PMD6/RE6)
- net D7: now also U1.60 (ERXD1/PMD0/RE0); no longer U1.3 (ETXD1/PMD7/RE7)
- net GND: now also U1.25 (VSS); no longer U1.9 (VSS)
- net PGEC1: no longer R4.1
- net PGED1: no longer R3.1
- net SW0: now also R12.2
- net SW1: now also R21.2
- net SW2: now also R23.2
- net SW3: now also R25.2
- net SW4: now also R11.2
- net SW5: now also R20.2
- net SW6: now also R22.2
- net SW7: now also R24.2
- net SCL4: no longer names the net of U1.6 (SCL4/SDO2/U3TX/PMA3/CN10/RG8)
- net SDA4: no longer names the net of U1.5 (SDA4/SDI2/U3RX/PMA4/CN9/RG7)
- net SW10: no longer names the net of U1.28 (TDI/AN13/PMA10/RB13)
- net SW10: no longer R22.2
- net SW11: no longer names the net of U1.30 (AN15/EMDC/AEMDC/OCFB/PMALL/PMA0/CN12/RB15)
- net SW11: no longer R23.2
- net SW12: no longer names the net of U1.47 (SOSCI/CN1/RC13)
- net SW12: no longer R24.2
- net SW13: no longer names the net of U1.37 (D+/RG2)
- net SW13: no longer R25.2
- net SW8: no longer names the net of U1.24 (TDO/AN11/PMA12/RB11)
- net SW8: now also R4.1; no longer R20.2
- net SW9: no longer names the net of U1.27 (TCK/AN12/PMA11/RB12)
- net SW9: now also R3.1; no longer R21.2
- net U1RX renamed OC3
- net U1TX renamed OC4
- no-connect marks 11 -> 19
