File: Chargeur Solaire/V0.10/Chargeur Solaire.sch (KiCad schematic (older format))
At the start: 36 parts, among them K1001 CONN_2, K1002 CONN_2, K1003 CONN_2, Q1001 BC557, Q1002 BUZ11, U1001 7805, U1002 TL072

Commit message: INIT
Parts:
- removed Q1002: BUZ11, Diodes_SMD:D-Pak_TO252AA, symbol BUZ11
- removed U1001: 7805, symbol 7805
- added P1001: CONN_01X06, f4deb-mod-library:KK-6-H, symbol CONN_01X06
- added Q1002: 34N06L, TO_SOT_Packages_SMD:TO-263-3Lead, symbol 34N06L
- added U1001: 7805-, TO_SOT_Packages_SMD:TO-252-2Lead, symbol 7805-
- C1001: footprint (none) -> Capacitors_Tantalum_SMD:Tantalum_Case-A_EIA-3216-18_Hand
- C1002, C1004: footprint (none) -> Capacitors_Tantalum_SMD:Tantalum_Case-B_EIA-3528-21_Hand
- D1001: footprint (none) -> Diodes_SMD:SMC_Handsoldering
- D1002, D1006: value 1n4148 -> LL4148; footprint (none) -> Diodes_SMD:MiniMELF_Standard
- D1007: value 1n5404 -> RS3K; footprint (none) -> Diodes_SMD:SMC_Standard
- K1001, K1002, K1003: footprint (none) -> Connectors_Phoenix:PhoenixContact_MC-GF_02x3.50mm_Angled_ThreadedFlange_MountHole
- RVAR1001: footprint (none) -> Potentiometers:Potentiometer_Trimmer-Suntan-TSR-3386C
- U1002: footprint (none) -> SMD_Packages:SOIC-8-N
Connections:
- net GND: now also P1001.1 (P1), Q1002.2 (D), U1001.2 (GND)
- net at C1003.1, R1003.1, U1002.2 (-): now also U1001.3 (VO)
- net at C1002.1, D1001.1 (K), Q1001.3 (E)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: now also U1001.1 (VI)
- net +BATT: now reaches C1004.1, D1001.2 (A), D1007.1 (K), K1001.2 (PM), K1002.2 (PM), R1001.1, R1013.1, R1016.1
- net +BATT: now also P1001.6 (P6)
- net at K1003.1 (P1), R1014.1, R1017.2: now also Q1002.3 (S)
- net at R1011.1, R1014.2: now also Q1002.1 (G)
- new net +12VA: P1001.5 (P5)
- new net +3V3: P1001.2 (P2)
- new net +5VA: P1001.4 (P4)
- new net +5VD: P1001.3 (P3)
Other:
- note added: "D1004 - Allumé -> Lumière faible\n Eteind -> Lumière forte\n"
- moved on the sheet: R1015
